File: pcb/pcb.kicad_pcb (KiCad board)
At the start: 2 copper layers, 53 x 29 mm, 30 parts, among them J4 Conn_02x05_Odd_Even, J5 RJ45_Amphenol_RJMG1BD3B8K1ANR, U1 ENC28J60x-SS, Y1 Crystal

Commit message: Mejoras en diseño
Other:
- board text added: "Modulo Ethernet Enc28j60 v.1.0 Esteva Santiago - FIUBA"
- board text added: "Tamaño de placa * 53 mm largo * 29 mm ancho Grilla: * 1 mm contorno PCB * 0.25 mm posicionamietno de componentes Tamaños seleccionados * 0,2 mm clearence * 0,25 mm ancho de pistas * 0,8 mm pad de via * 0,4 mm agujero de via Capas Top: F.Cu Botton: B.Cu"
